File: PCB/PedalPCB.kicad_sch (KiCad schematic)
At the start: 14 parts, among them J1 2x1, J2 Break, J3 Throttle, J4 SystemInput

Commit message: Add files via upload
Parts:
- H1, H2, H3, H4: footprint (none) -> MountingHole:MountingHole_4.3mm_M4
- J1: footprint CONN_S2B-PH-K-S_JST -> Connector_PinHeader_1.00mm:PinHeader_1x02_P1.00mm_Vertical
- J2, J3: footprint (none) -> Pedal:3pin
- J4: footprint (none) -> Pedal:JST4Pin
- R1, R2, R3, R4: footprint (none) -> Resistor_THT:R_Axial_DIN0204_L3.6mm_D1.6mm_P5.08mm_Horizontal
- U1: footprint ESP 32:ESP 32 BAJA -> Pedal:ESP 32 BAJA
- U2: footprint (none) -> Pedal:1x7 Connectors
Connections:
- net CanRX: now also U1.24 (D26); no longer U1.14 (D22)
- net CanTX: now also U1.25 (D27); no longer U1.11 (D21)
Changed lines of the file:
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@@
 	(wire
 		(pts
-			(xy 119.38 119.38) (xy 121.92 119.38)
+			(xy 148.59 99.06) (xy 149.86 99.06)
 		)
 		(stroke
@@
 	(wire
 		(pts
-			(xy 148.59 99.06) (xy 149.86 99.06)
+			(xy 93.98 96.52) (xy 99.06 96.52)
 		)
 		(stroke
@@
 	(wire
 		(pts
-			(xy 93.98 96.52) (xy 99.06 96.52)
+			(xy 166.37 152.4) (xy 168.91 152.4)
 		)
 		(stroke
@@
 	(wire
 		(pts
-			(xy 166.37 152.4) (xy 168.91 152.4)
+			(xy 147.32 118.11) (xy 149.86 118.11)
 		)
 		(stroke
@@
 	(wire
 		(pts
-			(xy 147.32 118.11) (xy 149.86 118.11)
+			(xy 143.51 102.87) (xy 149.86 102.87)
 		)
 		(stroke
@@
 	(wire
 		(pts
-			(xy 143.51 102.87) (xy 149.86 102.87)
+			(xy 158.75 138.43) (xy 158.75 142.24)
 		)
 		(stroke
@@
 	(wire
 		(pts
-			(xy 158.75 138.43) (xy 158.75 142.24)
+			(xy 97.79 99.06) (xy 99.06 99.06)
 		)
 		(stroke
@@
 	(wire
 		(pts
-			(xy 97.79 99.06) (xy 99.06 99.06)
+			(xy 158.75 123.19) (xy 158.75 129.54)
 		)
 		(stroke
@@
 	(wire
 		(pts
-			(xy 158.75 123.19) (xy 158.75 129.54)
+			(xy 119.38 137.16) (xy 121.92 137.16)
 		)
 		(stroke
@@
 	(wire
 		(pts
-			(xy 119.38 137.16) (xy 121.92 137.16)
+			(xy 93.98 99.06) (xy 97.79 99.06)
 		)
 		(stroke
@@
 	(wire
 		(pts
-			(xy 93.98 99.06) (xy 97.79 99.06)
+			(xy 166.37 129.54) (xy 168.91 129.54)
 		)
 		(stroke
@@
 	(wire
 		(pts
-			(xy 166.37 129.54) (xy 168.91 129.54)
+			(xy 143.51 106.68) (xy 149.86 106.68)
 		)
 		(stroke
@@
 	(wire
 		(pts
-			(xy 143.51 106.68) (xy 149.86 106.68)
+			(xy 119.38 129.54) (xy 120.65 129.54)
 		)
 		(stroke
@@
 	(wire
 		(pts
-			(xy 119.38 116.84) (xy 121.92 116.84)
+			(xy 119.38 127) (xy 120.65 127)
 		)
 		(stroke
@@
 		)
 	)
-	(label "Throttle"
-		(at 121.92 137.16 0)
+	(label "CanRX"
+		(at 120.65 127 0)
 		(fields_autoplaced yes)
 		(effects
@@
 		)
 	)
-	(label "CanL"
-		(at 166.37 154.94 180)
+	(label "CanTX"
+		(at 120.65 129.54 0)
 		(fields_autoplaced yes)
 		(effects
@@
 				(size 1.27 1.27)
 			)
-			(justify right bottom)
-		)
-	)
-	(label "CanTX"
-		(at 143.51 106.68 180)
+			(justify left bottom)
+		)
+	)
+	(label "Throttle"
+		(at 121.92 137.16 0)
 		(fields_autoplaced yes)
 		(effects
@@
 				(size 1.27 1.27)
 			)
-			(justify right bottom)
-		)
-	)
-	(label "CanH"
-		(at 147.32 114.3 180)
+			(justify left bottom)
+		)
+	)
+	(label "CanL"
+		(at 166.37 154.94 180)
 		(fields_autoplaced yes)
 		(effects
@@
 		)
 	)
-	(label "CanL"
-		(at 147.32 118.11 180)
+	(label "CanTX"
+		(at 143.51 106.68 180)
 		(fields_autoplaced yes)
 		(effects
@@
 		)
 	)
-	(label "CanRX"
-		(at 143.51 102.87 180)
+	(label "CanH"
+		(at 147.32 114.3 180)
 		(fields_autoplaced yes)
 		(effects
@@
 		)
 	)
-	(label "CanTX"
-		(at 121.92 116.84 0)
+	(label "CanL"
+		(at 147.32 118.11 180)
 		(fields_autoplaced yes)
 		(effects
@@
 				(size 1.27 1.27)
 			)
-			(justify left bottom)
+			(justify right bottom)
 		)
 	)
 	(label "CanRX"
-		(at 121.92 119.38 0)
+		(at 143.51 102.87 180)
 		(fields_autoplaced yes)
 		(effects
@@
 				(size 1.27 1.27)
 			)
-			(justify left bottom)
+			(justify right bottom)
 		)
 	)
@@
 			)
 		)
-		(property "Footprint" ""
+		(property "Footprint" "Resistor_THT:R_Axial_DIN0204_L3.6mm_D1.6mm_P5.08mm_Horizontal"
 			(at 162.56 127.762 90)
 			(effects
@@
 			)
 		)
-		(property "Footprint" ""
+		(property "Footprint" "MountingHole:MountingHole_4.3mm_M4"
 			(at 157.48 184.15 0)
 			(effects
@@
 			)
 		)
-		(property "Footprint" "ESP 32:ESP 32 BAJA"
+		(property "Footprint" "Pedal:ESP 32 BAJA"
 			(at 108.204 129.032 90)
 			(effects
@@
 			)
 		)
-		(property "Footprint" ""
+		(property "Footprint" "Resistor_THT:R_Axial_DIN0204_L3.6mm_D1.6mm_P5.08mm_Horizontal"
 			(at 162.56 140.462 90)
 			(effects
@@
 			)
 		)
-		(property "Footprint" ""
+		(property "Footprint" "Pedal:JST4Pin"
 			(at 173.99 152.4 0)
 			(effects
@@
 			)
 		)
-		(property "Footprint" ""
+		(property "Footprint" "MountingHole:MountingHole_4.3mm_M4"
 			(at 157.48 179.07 0)
 			(effects
@@
 			)
 		)
-		(property "Footprint" ""
+		(property "Footprint" "Pedal:1x7 Connectors"
 			(at 165.1 95.25 0)
 			(effects
@@
 			)
 		)
-		(property "Footprint" ""
+		(property "Footprint" "MountingHole:MountingHole_4.3mm_M4"
 			(at 157.48 194.31 0)
 			(effects
@@
 			)
 		)
-		(property "Footprint" ""
+		(property "Footprint" "Resistor_THT:R_Axial_DIN0204_L3.6mm_D1.6mm_P5.08mm_Horizontal"
 			(at 154.94 140.462 90)
 			(effects
@@
 			)
 		)
-		(property "Footprint" "CONN_S2B-PH-K-S_JST"
+		(property "Footprint" "Connector_PinHeader_1.00mm:PinHeader_1x02_P1.00mm_Vertical"
 			(at 140.97 74.93 0)
 			(effects
@@
 			)
 		)
-		(property "Footprint" ""
+		(property "Footprint" "MountingHole:MountingHole_4.3mm_M4"
 			(at 157.48 189.23 0)
 			(effects
@@
 			)
 		)
-		(property "Footprint" ""
+		(property "Footprint" "Pedal:3pin"
 			(at 173.99 125.73 0)
 			(effects
@@
 			)
 		)
-		(property "Footprint" ""
+		(property "Footprint" "Resistor_THT:R_Axial_DIN0204_L3.6mm_D1.6mm_P5.08mm_Horizontal"
 			(at 154.94 127.762 90)
 			(effects
@@
 			)
 		)
-		(property "Footprint" ""
+		(property "Footprint" "Pedal:3pin"
 			(at 173.99 138.43 0)
 			(effects

Commit message: Add files via upload
Connections:
- net CanTX: now also U1.23 (D25); no longer U1.25 (D27)
Changed lines of the file:
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@@
-	(wire
-		(pts
-			(xy 119.38 129.54) (xy 120.65 129.54)
-		)
-		(stroke
-			(width 0)
-			(type default)
-		)
-	)
 	(wire
 		(pts
@@
 		(pts
 			(xy 119.38 127) (xy 120.65 127)
+		)
+		(stroke
+			(width 0)
+			(type default)
+		)
+	)
+	(wire
+		(pts
+			(xy 119.38 124.46) (xy 120.65 124.46)
 		)
 		(stroke
@@
 		)
 	)
-	(label "CanTX"
-		(at 120.65 129.54 0)
-		(fields_autoplaced yes)
-		(effects
-			(font
-				(size 1.27 1.27)
-			)
-			(justify left bottom)
-		)
-	)
 	(label "Throttle"
 		(at 121.92 137.16 0)
@@
 		(fields_autoplaced yes)
 		(effects
+			(font
+				(size 1.27 1.27)
+			)
+			(justify left bottom)
+		)
+	)
+	(label "CanTX"
+		(at 120.65 124.46 0)
+		(fields_autoplaced yes)
+		(effects

Commit message: Add files via upload
Parts:
- removed J1: 2x1, Connector_PinHeader_1.00mm:PinHeader_1x02_P1.00mm_Vertical, symbol 2x1:S2B-PH-K-SLFSN
- added J5: Conn_01x04_Socket, Pedal:PowerBoard, symbol Connector:Conn_01x04_Socket
Connections:
- net +12V: now also J5.3 (12+)
- net +5V: now also J5.1 (+5v)
- net GND: now also J5.2 (GND), J5.4 (GND)
