File: PCB/PedalPCB.kicad_pcb (KiCad board)
At the start: 2 copper layers, 55 x 84.5 mm, 14 parts, among them J1 2x1, J2 Break, J3 Throttle, J4 SystemInput

Commit message: Add files via upload
Parts:
- moved H1 13.5 mm to (139.0, 126.5)
- moved J1 12.1 mm to (128.5, 121.0), turned to 90 degrees
- moved R4 9.59 mm to (141.5, 86.9), turned to -90 degrees
- moved R1 9.17 mm to (141.5, 99.0), turned to -90 degrees
- moved J2 8.51 mm to (146.5, 93.5)
- moved J3 8.51 mm to (146.0, 93.5)
- moved H2 7.83 mm to (143.0, 62.5)
- moved R3 6.78 mm to (138.5, 92.0), turned to 90 degrees
- moved R2 5.73 mm to (138.5, 104.0), turned to 90 degrees
Routing:
- net /Break: track 19.8 -> 11.1 mm
- net /Throttle: track 13.8 -> 7.54 mm
- net +5V: track 84.9 -> 79.1 mm
- net Net-(J2-Pin_1): track 3.95 -> 5.03 mm
- net /CanTX: track 32.2 -> 31.2 mm
- net Net-(J3-Pin_1): track 3.96 -> 4.93 mm
Other:
- board size 55 x 84.5 mm -> 45.5 x 84.5 mm

Commit message: Add files via upload
Parts:
- removed H4: MountingHole, MountingHole:MountingHole_4.3mm_M4
- removed J1: 2x1, Connector_PinHeader_1.00mm:PinHeader_1x02_P1.00mm_Vertical
- added J5: Conn_01x04_Socket, Pedal:PowerBoard, B.Cu at (135.5, 96.8)
- J4: moved to F.Cu
- moved J4 15.4 mm to (139.5, 55.0), turned to 0 degrees
- moved H1 10.9 mm to (142.0, 116.0)
- moved H2 1.58 mm to (143.5, 64.0)
- moved U1 0.10 mm to (121.2, 76.0)
Connections:
- U1 pad 23: unconnected-(U1-D25-Pad23) -> /CanTX
- U1 pad 25: /CanTX -> unconnected-(U1-D27-Pad25)
Routing:
- net +12V: track 0.00 -> 59.9 mm
- net /CanL: track 7.02 -> 32.3 mm
- net /CanH: track 7.02 -> 21.3 mm
- net GND: track 0.00 -> 8.99 mm
- net /CanTX: track 31.2 -> 36.1 mm
- net +5V: track 79.1 -> 77.4 mm
- net /CanRX: track 30.9 -> 31.3 mm, vias 1 -> 0
Other:
- board size 45.5 x 84.5 mm -> 45.5 x 73.5 mm
- board text added: "CanH"
- board text added: "CanL"
- board text added: "Rx"
- board text added: "TX"

Commit message: Update PCB to purchased version
Parts:
- added H1: MountingHole, MountingHole:MountingHole_4.3mm_M4, F.Cu at (111.0, 109.0)
- J5: moved to F.Cu
- moved J4 68.1 mm to (111.4, 117.0)
- moved U2 44.0 mm to (135.0, 106.0)
- moved J3 22.9 mm to (147.4, 70.6)
- moved R3 19.9 mm to (139.5, 72.1)
- moved R4 19.9 mm to (142.5, 67.0)
- moved R1 18.0 mm to (142.5, 81.0)
- moved R2 18.0 mm to (139.5, 86.0)
- moved U1 16.0 mm to (121.5, 60.0)
- moved J2 14.0 mm to (147.5, 79.5)
- moved J5 13.8 mm to (143.5, 85.5), turned to 0 degrees
- moved H2 9.12 mm to (145.0, 55.0)
- moved H1 2.55 mm to (144.5, 116.5)
- moved H3 2.55 mm to (111.0, 54.0)
Routing:
- net +3.3V: track 37.9 -> 58.4 mm
- net /CanL: track 32.3 -> 13.0 mm, vias 0 -> 1
- net +5V: track 77.4 -> 58.6 mm
- net +12V: track 59.9 -> 43.6 mm
- net GND: track 8.99 -> 0.00 mm
- net /CanH: track 21.3 -> 15.1 mm
- net Net-(J2-Pin_1): track 5.03 -> 8.06 mm
- net /Break: track 11.1 -> 14.0 mm
- net Net-(J3-Pin_1): track 4.93 -> 7.38 mm
- net /CanRX: track 31.3 -> 33.7 mm
- net /CanTX: track 36.1 -> 34.0 mm, vias 0 -> 1
- net /Throttle: track 7.54 -> 9.08 mm
Other:
- board text added: "+12V"
- board text added: "3.3V"
- board text added: "Brake"
- board text added: "CANH"
- board text added: "CANL"
- board text added: "HI"
- board text added: "LOW"
- board text added: "RX"
- board text added: "VCC"
- board text removed: "12+"
- board text removed: "Break"
- board text removed: "CanH"
- board text removed: "CanL"
- board text removed: "Rx"
